File: PCBs/HornPCB/Horn Circuit/Horn Circuit.kicad_pcb (KiCad board)
At the start: 2 copper layers, 100 x 91.7 mm, 20 parts, among them J1 Screw_Terminal_01x02 Speaker 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, J2 2301844-1, J4 2301844-1, U1 ESP32-S3-DevKitC, U2 DFR0299, U3 SN65HVD230DR

Commit message: Updated kicad project files for horn
Parts:
- added J3: Screw_Terminal_01x02 DAC OUT, TerminalBlock_Phoenix:TerminalBlock_Phoenix_MKDS-1,5-2-5.08_1x02_P5.08mm_Horizontal, F.Cu at (118.4, 66.0)
- added R5: 1K, Resistor_THT:R_Axial_DIN0207_L6.3mm_D2.5mm_P7.62mm_Horizontal, F.Cu at (112.0, 94.7)
- J1: footprint TerminalBlock_4Ucon:TerminalBlock_4Ucon_1x02_P3.50mm_Horizontal -> TerminalBlock_Phoenix:TerminalBlock_Phoenix_MKDS-1,5-2-5.08_1x02_P5.08mm_Horizontal
- JP1: value Jumper_2_Open -> Jumper_Term_Res
- moved R1 6.36 mm to (118.4, 94.8)
- moved D2 2.64 mm to (68.8, 86.0), turned to 0 degrees
- moved D1 2.51 mm to (69.1, 94.0), turned to 0 degrees
Connections:
- net /RX-SMD renamed CAN_RX
- net /TX-SMD renamed CAN_TX
- net Net-(J1-Pin_1) renamed /SPK+
- net Net-(J1-Pin_2) renamed /SPK-
- net Net-(U1-GPIO13/ADC2_CH2) renamed DFP BUSY
- D1 pad 1: Net-(D1-K) -> /STATUS LEDs-
- D1 pad 2: Net-(D1-A) -> /PREOP LED+
- D2 pad 1: Net-(D2-K) -> /STATUS LEDs-
- D2 pad 2: Net-(D1-A) -> /OP LED+
- R1 pad 1: Net-(U1-GPIO16/ADC2_CH5/32K_N) -> DFP_UART_TX
- R2 pad 1: Net-(D1-A) -> /STATUS LEDs-
- U1 pad 10: Net-(U1-GPIO17/ADC2_CH6) -> DFP_UART_TX
- U1 pad 11: unconnected-(U1-GPIO18/ADC2_CH7-Pad11) -> DFP_UART_RX
- U1 pad 4: Net-(D1-K) -> /PREOP LED+
- U1 pad 5: Net-(D2-K) -> /OP LED+
- U1 pad 9: Net-(U1-GPIO16/ADC2_CH5/32K_N) -> unconnected-(U1-GPIO16/ADC2_CH5/32K_N-Pad9)
- U2 pad 3: Net-(U1-GPIO17/ADC2_CH6) -> Net-(U2-TX)
- U2 pad 4: unconnected-(U2-DAC_R-Pad4) -> Net-(J3-Pin_2)
Routing:
- net Net-(D2-K): track 65.7 -> 0.00 mm
- net /OP LED+: track 0.00 -> 65.7 mm
- net Net-(D1-K): track 64.1 -> 0.00 mm
- net /PREOP LED+: track 0.00 -> 64.1 mm
- net Net-(D1-A): track 16.0 -> 0.00 mm
- net /STATUS LEDs-: track 0.00 -> 16.0 mm
- net DFP_UART_TX: track 0.00 -> 14.5 mm
- net Net-(U1-GPIO17/ADC2_CH6): track 13.5 -> 0.00 mm
- net DFP_UART_RX: track 0.00 -> 10.8 mm
- net Net-(U2-RX): track 16.9 -> 27.0 mm
- net Net-(U1-GPIO16/ADC2_CH5/32K_N): track 8.41 -> 0.00 mm
- net Net-(U2-TX): track 0.00 -> 7.98 mm
- net /SPK-: track 36.0 -> 36.6 mm
Other:
- board text added: "23/APR/26 V2.1"
- board text removed: "16/MAR/26 V2.0"

Commit message: DFPlayer DAC_R outputs
Parts:
- removed J1: Screw_Terminal_01x02 Speaker Out, TerminalBlock_Phoenix:TerminalBlock_Phoenix_MKDS-1,5-2-5.08_1x02_P5.08mm_Horizontal
- moved J3 45.9 mm to (72.7, 69.6)
Connections:
- net Net-(J3-Pin_2) renamed /DAC_R+
- U2 pad 6: /SPK- -> unconnected-(U2-SPK1-Pad6)
- U2 pad 8: /SPK+ -> unconnected-(U2-SPK2-Pad8)
Routing:
- net /DAC_R+: track 0.00 -> 37.3 mm
- net /SPK-: track 36.6 -> 0.00 mm
- net /SPK+: track 35.3 -> 0.00 mm
- net Net-(U2-RX): track 27.0 -> 15.4 mm
Other:
- board text added: "29/APR/26 V2.2"
- board text removed: "23/APR/26 V2.1"
